File: HW/Robot/Servo_Current_Limiter/substracter.kicad_sch (KiCad schematic)
At the start: 5 parts, among them J3 1x1 2.54mm male

Commit message: Sch update.
Parts:
- added U1: LM324, Package_DIP:DIP-14_W7.62mm, symbol Amplifier_Operational:LM324
- R21: renamed from R3; value 220k -> 100k
- R22: renamed from R4; value 220k -> 10k
- R23: renamed from R5; value 220k -> 10k
- R24: renamed from R6; value 220k -> 100k; footprint For_Rasterboard:R_Axial_DIN0207_L6.3mm_D2.5mm_Pinf_Horizontal -> For_Rasterboard:R_Axial_DIN0207_L6.3mm_D2.5mm_P2.54mm_Vertical
- renumbered J3 to J14
Connections:
- net OUT: now also U1.14
- net GNDA renamed GND
- net op/IN+: no longer names the net of R21.2, R22.2
- net op/IN+: now also U1.12 (+)
- net op/IN-: no longer names the net of R23.1, R24.2
- net op/IN-: now also U1.13 (-)
Other:
- removed sheet op
Changed lines of the file:
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@@
     (stroke (width 0) (type default) (color 0 0 0 0))
   )
-  (wire (pts (xy 185.42 81.28) (xy 190.5 81.28))
+  (wire (pts (xy 179.07 81.28) (xy 190.5 81.28))
     (stroke (width 0) (type default) (color 0 0 0 0))
   )
@@
     (effects (font (size 1.27 1.27)) (justify left))
   )
-  (symbol (lib_id "Connector:TestPoint") (at 207.01 78.74 0) (unit 1)
-    (in_bom yes) (on_board yes)
-    (property "Reference" "J3" (id 0) (at 207.01 69.85 0))
-    (property "Value" "1x1 2.54mm male" (id 1) (at 207.01 72.39 0))
-    (property "Footprint" "Connector_PinHeader_2.54mm:PinHeader_1x01_P2.54mm_Vertical" (id 2) (at 207.01 78.74 0)
+  (symbol (lib_id "power:GND") (at 132.08 71.12 270) (unit 1)
+    (in_bom yes) (on_board yes) (fields_autoplaced)
+    (property "Reference" "#PWR?" (id 0) (at 125.73 71.12 0)
       (effects (font (size 1.27 1.27)) hide)
     )
-    (property "Datasheet" "~" (id 3) (at 207.01 78.74 0)
-      (effects (font (size 1.27 1.27)) hide)
-    )
-    (pin "1")
-  )
-  (symbol (lib_id "power:GNDA") (at 132.08 71.12 270) (unit 1)
-    (in_bom yes) (on_board yes) (fields_autoplaced)
-    (property "Reference" "#PWR07" (id 0) (at 125.73 71.12 0)
-      (effects (font (size 1.27 1.27)) hide)
-    )
-    (property "Value" "GNDA" (id 1) (at 128.27 71.1199 90)
+    (property "Value" "GND" (id 1) (at 128.905 71.1199 90)
       (effects (font (size 1.27 1.27)) (justify right))
     )
@@
     (pin "1")
   )
+  (symbol (lib_id "Connector:TestPoint") (at 207.01 78.74 0) (unit 1)
+    (in_bom yes) (on_board yes)
+    (property "Reference" "J14" (id 0) (at 207.01 69.85 0))
+    (property "Value" "1x1 2.54mm male" (id 1) (at 207.01 72.39 0))
+    (property "Footprint" "Connector_PinHeader_2.54mm:PinHeader_1x01_P2.54mm_Vertical" (id 2) (at 207.01 78.74 0)
+      (effects (font (size 1.27 1.27)) hide)
+    )
+    (property "Datasheet" "~" (id 3) (at 207.01 78.74 0)
+      (effects (font (size 1.27 1.27)) hide)
+    )
+    (pin "1")
+  )
+  (symbol (lib_id "Amplifier_Operational:LM324") (at 171.45 81.28 0) (unit 4)
+    (in_bom yes) (on_board yes) (fields_autoplaced)
+    (property "Reference" "U1" (id 0) (at 171.45 70.485 0))
+    (property "Value" "LM324" (id 1) (at 171.45 73.025 0))
+    (property "Footprint" "Package_DIP:DIP-14_W7.62mm" (id 2) (at 170.18 78.74 0)
+      (effects (font (size 1.27 1.27)) hide)
+    )
+    (property "Datasheet" "http://www.ti.com/lit/ds/symlink/lm2902-n.pdf" (id 3) (at 172.72 76.2 0)
+      (effects (font (size 1.27 1.27)) hide)
+    )
+    (pin "1")
+    (pin "2")
+    (pin "3")
+    (pin "5")
+    (pin "6")
+    (pin "7")
+    (pin "10")
+    (pin "8")
+    (pin "9")
+    (pin "12")
+    (pin "13")
+    (pin "14")
+    (pin "11")
+    (pin "4")
+  )
   (symbol (lib_id "Device:R") (at 146.05 83.82 270) (mirror x) (unit 1)
     (in_bom yes) (on_board yes)
-    (property "Reference" "R5" (id 0) (at 146.05 89.0778 90))
-    (property "Value" "220k" (id 1) (at 146.05 86.7664 90))
+    (property "Reference" "R23" (id 0) (at 146.05 89.0778 90))
+    (property "Value" "10k" (id 1) (at 146.05 86.7664 90))
     (property "Footprint" "For_Rasterboard:R_Axial_DIN0207_L6.3mm_D2.5mm_P7.62mm_Horizontal" (id 2) (at 146.05 85.598 90)
       (effects (font (size 1.27 1.27)) hide)
@@
   (symbol (lib_id "Device:R") (at 167.64 99.06 270) (unit 1)
     (in_bom yes) (on_board yes)
-    (property "Reference" "R6" (id 0) (at 167.64 93.8022 90))
-    (property "Value" "220k" (id 1) (at 167.64 96.1136 90))
-    (property "Footprint" "For_Rasterboard:R_Axial_DIN0207_L6.3mm_D2.5mm_Pinf_Horizontal" (id 2) (at 167.64 97.282 90)
+    (property "Reference" "R24" (id 0) (at 167.64 93.8022 90))
+    (property "Value" "100k" (id 1) (at 167.64 96.1136 90))
+    (property "Footprint" "For_Rasterboard:R_Axial_DIN0207_L6.3mm_D2.5mm_P2.54mm_Vertical" (id 2) (at 167.64 97.282 90)
       (effects (font (size 1.27 1.27)) hide)
     )
@@
   (symbol (lib_id "Device:R") (at 146.05 71.12 90) (mirror x) (unit 1)
     (in_bom yes) (on_board yes)
-    (property "Reference" "R3" (id 0) (at 146.05 65.8622 90))
-    (property "Value" "220k" (id 1) (at 146.05 68.1736 90))
+    (property "Reference" "R21" (id 0) (at 146.05 65.8622 90))
+    (property "Value" "100k" (id 1) (at 146.05 68.1736 90))
     (property "Footprint" "For_Rasterboard:R_Axial_DIN0207_L6.3mm_D2.5mm_Pinf_Horizontal" (id 2) (at 146.05 69.342 90)
       (effects (font (size 1.27 1.27)) hide)
@@
   (symbol (lib_id "Device:R") (at 146.05 78.74 90) (mirror x) (unit 1)
     (in_bom yes) (on_board yes)
-    (property "Reference" "R4" (id 0) (at 146.05 73.4822 90))
-    (property "Value" "220k" (id 1) (at 146.05 75.7936 90))
+    (property "Reference" "R22" (id 0) (at 146.05 73.4822 90))
+    (property "Value" "10k" (id 1) (at 146.05 75.7936 90))
     (property "Footprint" "For_Rasterboard:R_Axial_DIN0207_L6.3mm_D2.5mm_P7.62mm_Horizontal" (id 2) (at 146.05 76.962 90)
       (effects (font (size 1.27 1.27)) hide)
@@
     (pin "2")
   )
-  (sheet (at 163.83 77.47) (size 21.59 7.62) (fields_autoplaced)
-    (stroke (width 0.1524) (type solid) (color 0 0 0 0))
-    (fill (color 0 0 0 0.0000))
-    (property "Sheet name" "op" (id 0) (at 163.83 76.7584 0)
-      (effects (font (size 1.27 1.27)) (justify left bottom))
-    )
-    (property "Sheet file" "op_amp.kicad_sch" (id 1) (at 163.83 85.6746 0)
-      (effects (font (size 1.27 1.27)) (justify left top))
-    )
-    (pin "OUT" output (at 185.42 81.28 0)
-      (effects (font (size 1.27 1.27)) (justify right))
-    )
-    (pin "IN+" input (at 163.83 78.74 180)
-      (effects (font (size 1.27 1.27)) (justify left))
-    )
-    (pin "IN-" input (at 163.83 83.82 180)
-      (effects (font (size 1.27 1.27)) (justify left))
-    )
-  )
 )

Commit message: Working.
Parts:
- R23: footprint For_Rasterboard:R_Axial_DIN0207_L6.3mm_D2.5mm_P7.62mm_Horizontal -> Resistor_THT:R_Axial_DIN0207_L6.3mm_D2.5mm_P10.16mm_Horizontal
Changed lines of the file:
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@@
   (symbol (lib_id "power:GND") (at 132.08 71.12 270) (unit 1)
     (in_bom yes) (on_board yes) (fields_autoplaced)
-    (property "Reference" "#PWR?" (id 0) (at 125.73 71.12 0)
+    (property "Reference" "#PWR0101" (id 0) (at 125.73 71.12 0)
       (effects (font (size 1.27 1.27)) hide)
     )
@@
     (property "Reference" "R23" (id 0) (at 146.05 89.0778 90))
     (property "Value" "10k" (id 1) (at 146.05 86.7664 90))
-    (property "Footprint" "For_Rasterboard:R_Axial_DIN0207_L6.3mm_D2.5mm_P7.62mm_Horizontal" (id 2) (at 146.05 85.598 90)
+    (property "Footprint" "Resistor_THT:R_Axial_DIN0207_L6.3mm_D2.5mm_P10.16mm_Horizontal" (id 2) (at 146.05 85.598 90)
       (effects (font (size 1.27 1.27)) hide)
     )
