File: HW/Robot/Servo_Current_Limiter/Servo_Current_Limiter.kicad_pcb (KiCad board)
At the start: 2 copper layers, 54 parts, among them J1 1x3 2.54mm male, J10 1x3 2.54mm male, J11 1x1 2.54mm male, J12 1x1 2.54mm male, J13 1x3 2.54mm male, J14 1x1 2.54mm male, J2 Conn_02x05_Odd_Even, J3 1x1 2.54mm male, J4 1x3 2.54mm male, J5 1x1 2.54mm male, J6 1x1 2.54mm male, J7 1x3 2.54mm male, J8 1x1 2.54mm male, J9 1x1 2.54mm male, Q1 IRF4905, Q2 BC548, Q3 IRF4905, Q4 BC548, Q5 IRF4905, Q6 BC548, Q7 IRF4905, Q8 BC548, U1 LM324

Commit message: Correction.
Parts:
- C1: footprint For_Rasterboard:C_Disc_D3.0mm_W1.6mm_P5.00mm -> For_Rasterboard:C_Disc_D3.0mm_W1.6mm_P2.50mm
- R4: footprint For_Rasterboard:R_Axial_DIN0207_L6.3mm_D2.5mm_P5.08mm_Vertical -> For_Rasterboard:R_Axial_DIN0207_L6.3mm_D2.5mm_P12.70mm_Horizontal
- R5: footprint Resistor_THT:R_Axial_DIN0207_L6.3mm_D2.5mm_P10.16mm_Horizontal -> For_Rasterboard:R_Axial_DIN0207_L6.3mm_D2.5mm_P2.54mm_Vertical
- moved R4 9.20 mm to (71.1, 167.4)
- moved R5 5.08 mm to (66.0, 177.6)
Connections:
- R10 pad 1: /ch1/N -> /ch1/P
- R11 pad 2: /ch1/P -> /ch1/N
- R16 pad 1: /ch2/N -> /ch2/P
- R17 pad 2: /ch2/P -> /ch2/N
- R22 pad 1: /ch3/N -> /ch3/P
- R23 pad 2: /ch3/P -> /ch3/N
- R4 pad 1: /ch0/N -> /ch0/P
- R5 pad 2: /ch0/P -> /ch0/N
Routing:
- net Net-(R5-Pad1): track 33.0 -> 38.1 mm
