File: HW/Robot/Servo_Current_Limiter/channel.kicad_sch (KiCad schematic)
At the start: 7 parts, among them J1 1x1 2.54mm male, J2 1x5 2.54mm male, Q1 IRF4905, Q2 BC338

Commit message: Sch update.
Parts:
- removed J2: 1x5 2.54mm male, Connector_PinSocket_2.54mm:PinSocket_1x05_P2.54mm_Vertical, symbol Connector_Generic:Conn_01x05
- added J13: 1x3 2.54mm male, Connector_PinHeader_2.54mm:PinHeader_1x03_P2.54mm_Vertical, symbol Connector_Generic:Conn_01x03
- renumbered J1 to J12, Q1 to Q7, Q2 to Q8, R1 to R19, R2 to R20, RV1 to RV4
Connections:
- net GND: now also J13.1 (Pin_1)
- net N: now also J13.2 (Pin_2)
- net PWM: now also J13.3 (Pin_3)
Changed lines of the file:
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@@
     (effects (font (size 1.27 1.27)) (justify right bottom))
+  )
+  (hierarchical_label "PWM" (shape input) (at 228.6 48.26 180)
+    (effects (font (size 1.27 1.27)) (justify right))
   )
   (hierarchical_label "DISABLE" (shape input) (at 121.92 53.34 180)
@@
   (symbol (lib_id "power:+5V") (at 140.97 66.04 0) (unit 1)
     (in_bom yes) (on_board yes) (fields_autoplaced)
-    (property "Reference" "#PWR01" (id 0) (at 140.97 69.85 0)
+    (property "Reference" "#PWR026" (id 0) (at 140.97 69.85 0)
       (effects (font (size 1.27 1.27)) hide)
     )
@@
   (symbol (lib_id "power:+5V") (at 168.91 41.91 90) (unit 1)
     (in_bom yes) (on_board yes)
-    (property "Reference" "#PWR05" (id 0) (at 172.72 41.91 0)
+    (property "Reference" "#PWR028" (id 0) (at 172.72 41.91 0)
       (effects (font (size 1.27 1.27)) hide)
     )
@@
   (symbol (lib_id "Connector:TestPoint") (at 160.02 80.01 0) (unit 1)
     (in_bom yes) (on_board yes)
-    (property "Reference" "J1" (id 0) (at 160.02 71.12 0))
+    (property "Reference" "J12" (id 0) (at 160.02 71.12 0))
     (property "Value" "1x1 2.54mm male" (id 1) (at 160.02 73.66 0))
     (property "Footprint" "Connector_PinHeader_2.54mm:PinHeader_1x01_P2.54mm_Vertical" (id 2) (at 160.02 80.01 0)
@@
   (symbol (lib_id "Device:R") (at 140.97 72.39 0) (unit 1)
     (in_bom yes) (on_board yes)
-    (property "Reference" "R1" (id 0) (at 135.7122 72.39 90))
+    (property "Reference" "R19" (id 0) (at 135.7122 72.39 90))
     (property "Value" "220" (id 1) (at 138.0236 72.39 90))
     (property "Footprint" "For_Rasterboard:R_Axial_DIN0207_L6.3mm_D2.5mm_Pinf_Horizontal" (id 2) (at 139.192 72.39 90)
@@
   (symbol (lib_id "Device:Q_PMOS_GDS") (at 177.8 44.45 270) (mirror x) (unit 1)
     (in_bom yes) (on_board yes)
-    (property "Reference" "Q1" (id 0) (at 177.8 35.7632 90))
+    (property "Reference" "Q7" (id 0) (at 177.8 35.7632 90))
     (property "Value" "IRF4905" (id 1) (at 177.8 38.0746 90))
     (property "Footprint" "Package_TO_SOT_THT:TO-220-3_Vertical" (id 2) (at 180.34 39.37 0)
@@
   (symbol (lib_id "Servo_Current_Limiter-cache:BC338") (at 180.34 77.47 0) (mirror y) (unit 1)
     (in_bom yes) (on_board yes) (fields_autoplaced)
-    (property "Reference" "Q2" (id 0) (at 175.26 76.1999 0)
+    (property "Reference" "Q8" (id 0) (at 175.26 76.1999 0)
       (effects (font (size 1.27 1.27)) (justify left))
     )
@@
   (symbol (lib_id "power:GND") (at 140.97 90.17 0) (mirror y) (unit 1)
     (in_bom yes) (on_board yes)
-    (property "Reference" "#PWR04" (id 0) (at 140.97 96.52 0)
+    (property "Reference" "#PWR027" (id 0) (at 140.97 96.52 0)
       (effects (font (size 1.27 1.27)) hide)
     )
@@
   (symbol (lib_id "Device:R_Potentiometer") (at 140.97 82.55 0) (unit 1)
     (in_bom yes) (on_board yes) (fields_autoplaced)
-    (property "Reference" "RV1" (id 0) (at 138.43 81.2799 0)
+    (property "Reference" "RV4" (id 0) (at 138.43 81.2799 0)
       (effects (font (size 1.27 1.27)) (justify right))
     )
@@
   (symbol (lib_id "Device:R") (at 191.77 41.91 270) (unit 1)
     (in_bom yes) (on_board yes)
-    (property "Reference" "R2" (id 0) (at 191.77 36.6522 90))
+    (property "Reference" "R20" (id 0) (at 191.77 36.6522 90))
     (property "Value" "0.1" (id 1) (at 191.77 38.9636 90))
     (property "Footprint" "Resistor_THT:R_Axial_DIN0207_L6.3mm_D2.5mm_P10.16mm_Horizontal" (id 2) (at 191.77 40.132 90)
@@
   (symbol (lib_id "power:GND") (at 231.775 53.34 270) (unit 1)
     (in_bom yes) (on_board yes) (fields_autoplaced)
-    (property "Reference" "#PWR06" (id 0) (at 225.425 53.34 0)
+    (property "Reference" "#PWR029" (id 0) (at 225.425 53.34 0)
       (effects (font (size 1.27 1.27)) hide)
     )
@@
     (pin "1")
   )
-  (symbol (lib_id "Connector_Generic:Conn_01x05") (at 238.76 48.26 0) (unit 1)
+  (symbol (lib_id "Connector_Generic:Conn_01x03") (at 238.76 50.8 0) (mirror x) (unit 1)
     (in_bom yes) (on_board yes)
-    (property "Reference" "J2" (id 0) (at 236.22 39.37 0)
+    (property "Reference" "J13" (id 0) (at 241.935 52.0701 0)
       (effects (font (size 1.27 1.27)) (justify left))
     )
-    (property "Value" "1x5 2.54mm male" (id 1) (at 226.06 36.83 0)
+    (property "Value" "1x3 2.54mm male" (id 1) (at 241.935 49.5301 0)
       (effects (font (size 1.27 1.27)) (justify left))
     )
-    (property "Footprint" "Connector_PinSocket_2.54mm:PinSocket_1x05_P2.54mm_Vertical" (id 2) (at 238.76 48.26 0)
+    (property "Footprint" "Connector_PinHeader_2.54mm:PinHeader_1x03_P2.54mm_Vertical" (id 2) (at 238.76 50.8 0)
       (effects (font (size 1.27 1.27)) hide)
     )
-    (property "Datasheet" "~" (id 3) (at 238.76 48.26 0)
+    (property "Datasheet" "~" (id 3) (at 238.76 50.8 0)
       (effects (font (size 1.27 1.27)) hide)
     )
-    (property "Comment" "To Servo Motor" (id 4) (at 238.76 31.75 0))
+    (property "Comment" "To Servo" (id 4) (at 246.38 55.88 0))
     (pin "1")
     (pin "2")
     (pin "3")
-    (pin "4")
-    (pin "5")
   )
   (sheet (at 214.63 69.85) (size 16.51 15.24) (fields_autoplaced)

Commit message: Working.
Parts:
- removed Q8: BC338, For_Rasterboard:TO-92_Inline_inf, symbol Servo_Current_Limiter-cache:BC338
- added Q2: BC548, For_Rasterboard:TO-92_Inline_inf, symbol Servo_Current_Limiter-cache:BC548
- R20: footprint Resistor_THT:R_Axial_DIN0207_L6.3mm_D2.5mm_P10.16mm_Horizontal -> For_Rasterboard:R_Axial_DIN0207_L6.3mm_D2.5mm_P7.62mm_Horizontal
Connections:
- net DISABLE: now also Q2.1 (C)
- net OUT: now also Q2.2 (B)
- net at J12.1, RV4.2: now also Q2.3 (E)
Changed lines of the file:
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@@
     (pin "2")
+  )
+  (symbol (lib_id "Servo_Current_Limiter-cache:BC548") (at 180.34 77.47 0) (mirror y) (unit 1)
+    (in_bom yes) (on_board yes) (fields_autoplaced)
+    (property "Reference" "Q2" (id 0) (at 175.26 76.1999 0)
+      (effects (font (size 1.27 1.27)) (justify left))
+    )
+    (property "Value" "BC548" (id 1) (at 175.26 78.7399 0)
+      (effects (font (size 1.27 1.27)) (justify left))
+    )
+    (property "Footprint" "For_Rasterboard:TO-92_Inline_inf" (id 2) (at 175.26 79.375 0)
+      (effects (font (size 1.27 1.27) italic) (justify left) hide)
+    )
+    (property "Datasheet" "" (id 3) (at 180.34 77.47 0)
+      (effects (font (size 1.27 1.27)) (justify left) hide)
+    )
+    (pin "1")
+    (pin "2")
+    (pin "3")
   )
   (symbol (lib_id "Device:Q_PMOS_GDS") (at 177.8 44.45 270) (mirror x) (unit 1)
@@
     (property "Datasheet" "~" (id 3) (at 177.8 44.45 0)
       (effects (font (size 1.27 1.27)) hide)
-    )
-    (pin "1")
-    (pin "2")
-    (pin "3")
-  )
-  (symbol (lib_id "Servo_Current_Limiter-cache:BC338") (at 180.34 77.47 0) (mirror y) (unit 1)
-    (in_bom yes) (on_board yes) (fields_autoplaced)
-    (property "Reference" "Q8" (id 0) (at 175.26 76.1999 0)
-      (effects (font (size 1.27 1.27)) (justify left))
-    )
-    (property "Value" "BC338" (id 1) (at 175.26 78.7399 0)
-      (effects (font (size 1.27 1.27)) (justify left))
-    )
-    (property "Footprint" "For_Rasterboard:TO-92_Inline_inf" (id 2) (at 175.26 79.375 0)
-      (effects (font (size 1.27 1.27) italic) (justify left) hide)
-    )
-    (property "Datasheet" "" (id 3) (at 180.34 77.47 0)
-      (effects (font (size 1.27 1.27)) (justify left) hide)
     )
     (pin "1")
@@
     (property "Reference" "R20" (id 0) (at 191.77 36.6522 90))
     (property "Value" "0.1" (id 1) (at 191.77 38.9636 90))
-    (property "Footprint" "Resistor_THT:R_Axial_DIN0207_L6.3mm_D2.5mm_P10.16mm_Horizontal" (id 2) (at 191.77 40.132 90)
+    (property "Footprint" "For_Rasterboard:R_Axial_DIN0207_L6.3mm_D2.5mm_P7.62mm_Horizontal" (id 2) (at 191.77 40.132 90)
       (effects (font (size 1.27 1.27)) hide)
     )

Commit message: PCB for 1 channel done.
Parts:
- renumbered Q2 to Q8
Changed lines of the file:
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@@
   (symbol (lib_id "Servo_Current_Limiter-cache:BC548") (at 180.34 77.47 0) (mirror y) (unit 1)
     (in_bom yes) (on_board yes) (fields_autoplaced)
-    (property "Reference" "Q2" (id 0) (at 175.26 76.1999 0)
+    (property "Reference" "Q8" (id 0) (at 175.26 76.1999 0)
       (effects (font (size 1.27 1.27)) (justify left))
     )

Commit message: Correction.
Connections:
- net OUT: now also Q8.3 (E); no longer Q8.2 (B)
- net at J12.1, RV4.2: now also Q8.2 (B); no longer Q8.3 (E)
Other:
- moved on the sheet: J12, J13, Q7, Q8, R19, R20, RV4

Commit message: Correction.
Changed lines of the file:
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@@
     (effects (font (size 1.27 1.27)) (justify left bottom))
   )
-  (label "N" (at 255.905 78.74 180)
+  (label "N" (at 255.905 83.82 180)
     (effects (font (size 1.27 1.27)) (justify right bottom))
   )
-  (label "P" (at 255.905 83.82 180)
+  (label "P" (at 255.905 78.74 180)
     (effects (font (size 1.27 1.27)) (justify right bottom))
   )
